File: pcb/source/keyboardv2.kicad_pcb (KiCad board)
At the start: 2 copper layers, 406.7 x 100.5 mm, 147 parts, among them J1 AudioJack4, J2 AudioJack4, SW1 SW_Push, SW10 SW_Push, SW11 SW_Push, SW12 SW_Push, SW13 SW_Push, SW14 SW_Push, SW15 SW_Push, SW16 SW_Push, SW17 SW_Push, SW18 SW_Push, SW19 SW_Push, SW2 SW_Push, SW20 SW_Push, SW21 SW_Push, SW22 SW_Push, SW23 SW_Push, SW24 SW_Push, SW25 SW_Push, SW26 SW_Push, SW27 SW_Push, SW28 SW_Push, SW29 SW_Push, SW3 SW_Push, SW30 SW_Push, SW31 SW_Push, SW32 SW_Push, SW33 SW_Push, SW34 SW_Push, SW35 SW_Push, SW36 SW_Push, SW37 SW_Push, SW38 SW_Push, SW39 SW_Push, SW4 SW_Push, SW40 SW_Push, SW41 SW_Push, SW42 SW_Push, SW43 SW_Push, SW44 SW_Push, SW45 SW_Push, SW46 SW_Push, SW47 SW_Push, SW48 SW_Push, SW49 SW_Push, SW5 SW_Push, SW50 SW_Push, SW51 SW_Push, SW52 SW_Push, SW53 SW_Push, SW54 SW_Push, SW55 SW_Push, SW56 SW_Push, SW57 SW_Push, SW58 SW_Push, SW59 SW_Push, SW6 SW_Push, SW60 SW_Push, SW61 SW_Push, SW62 SW_Push, SW63 SW_Push, SW64 SW_Push, SW65 SW_Push, SW66 SW_Push, SW67 SW_Push, SW68 SW_Push, SW69 SW_Push, SW7 SW_Push, SW8 SW_Push, SW9 SW_Push

Commit message: minor updates with bom added
Parts:
- removed hfscjkzhslfjk, logo1, logo2: LOGO, LOGO
- moved A1 27.9 mm to (232.7, 65.9)
- moved D16 27.9 mm to (131.9, 103.5)
- moved D18 27.9 mm to (170.0, 103.5)
- moved D20 27.9 mm to (208.1, 103.4)
- moved D3 27.9 mm to (146.2, 84.4)
- moved D30 27.9 mm to (136.6, 122.5)
- moved D32 27.9 mm to (174.7, 122.5)
- moved D34 27.9 mm to (212.8, 122.5)
- moved D44 27.9 mm to (160.5, 141.6)
- moved D45 27.9 mm to (179.5, 141.6)
- moved D47 27.9 mm to (217.6, 141.6)
- moved D5 27.9 mm to (184.3, 84.4)
- moved D6 27.9 mm to (203.4, 84.4)
- moved SW17 27.9 mm to (147.1, 95.3)
- moved SW19 27.9 mm to (185.2, 95.3)
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Routing:
- net Net-(A3-GPIO6): track 242.4 -> 220.1 mm, vias 2 -> 1
- net Net-(A1-GPIO1): track 275.6 -> 259.9 mm, vias 2 -> 3
- net Net-(A3-GPIO11): track 222.7 -> 210.6 mm
- net Net-(A3-GPIO19): track 30.2 -> 41.7 mm, vias 2 -> 1
- net Net-(A1-GPIO3): track 281.0 -> 291.5 mm, vias 3 -> 4
- net Net-(A1-GPIO0): track 260.6 -> 251.7 mm, vias 2 -> 1
- net Net-(A3-GPIO10): track 199.0 -> 192.2 mm
- net Net-(A1-GPIO19): track 30.1 -> 24.7 mm, vias 2 -> 0
- net Net-(A1-GPIO5): track 108.4 -> 103.6 mm
- net Net-(A3-GPIO1): track 124.9 -> 129.3 mm, vias 2 -> 1
- net Net-(A3-3V3): track 52.8 -> 57.1 mm
- net Net-(A3-GPIO12): track 228.5 -> 232.6 mm
- net Net-(A1-GPIO2): track 263.4 -> 259.9 mm
- net Net-(A1-GPIO8): track 137.9 -> 141.1 mm
- net Net-(A1-GPIO10): track 157.1 -> 159.5 mm
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Other:
- board size 406.7 x 100.5 mm -> 364.2 x 100.5 mm
