File: pcb/keyboardv2.kicad_sch (KiCad schematic)
At the start: 75 parts, among them J2 AudioJack4, SW10 SW_Push, SW11 SW_Push, SW12 SW_Push, SW13 SW_Push, SW14 SW_Push, SW21 SW_Push, SW22 SW_Push, SW23 SW_Push, SW24 SW_Push, SW25 SW_Push, SW26 SW_Push, SW27 SW_Push, SW28 SW_Push, SW35 SW_Push, SW36 SW_Push, SW37 SW_Push, SW38 SW_Push, SW39 SW_Push, SW40 SW_Push, SW41 SW_Push, SW48 SW_Push, SW49 SW_Push, SW50 SW_Push, SW51 SW_Push, SW52 SW_Push, SW53 SW_Push, SW54 SW_Push, SW59 SW_Push, SW60 SW_Push, SW61 SW_Push, SW62 SW_Push, SW63 SW_Push, SW64 SW_Push, SW65 SW_Push, SW8 SW_Push, SW9 SW_Push

Commit message: bom changes and layout changes
Parts:
- removed A3: RaspberryPi_Pico, Module:RaspberryPi_Pico_Common_THT, symbol MCU_Module_RaspberryPi_Pico:RaspberryPi_Pico
- removed D10, D11, D12, D13, D14, D21, D22, D23, D24, D25, D26, D27, D28, D35, D36, D37, D38, D39, D40, D41, D48, D49, D50, D51, D52, D53, D54, D59, D60, D61, D62, D63, D64, D65, D8, D9: 1N4148, Diode_THT:D_DO-35_SOD27_P7.62mm_Horizontal, symbol Diode:1N4148
- removed J2: AudioJack4, Library:TENSILITY_54-00174, symbol Connector_Audio:AudioJack4_SwitchT1
- removed SW10, SW11, SW12, SW13, SW21, SW22, SW23, SW24, SW25, SW26, SW27, SW28, SW35, SW36, SW37, SW38, SW39, SW40, SW48, SW49, SW50, SW51, SW52, SW54, SW60, SW61, SW62, SW63, SW64, SW65, SW8, SW9: SW_Push, MX_Hotswap:MX-Hotswap-1U, symbol Switch:SW_Push
- removed SW14, SW41: SW_Push, MX_Hotswap:MX-Hotswap-1.75U, symbol Switch:SW_Push
- removed SW53: SW_Push, MX_Hotswap:MX-Hotswap-1.25U, symbol Switch:SW_Push
- removed SW59: SW_Push, MX_Hotswap:MX-Hotswap-2U, symbol Switch:SW_Push
- removed U2: ~, Library:SSD1306-0.91-OLED-4pin-128x32, symbol display:.91{dblquote}_4-pin_OLED
- added A1: RaspberryPi_Pico, Module:RaspberryPi_Pico_Common_THT, symbol MCU_Module_RaspberryPi_Pico:RaspberryPi_Pico
- added D1, D15, D16, D17, D18, D19, D2, D20, D29, D3, D30, D31, D32, D33, D34, D4, D42, D43, D44, D45, D46, D47, D5, D55, D56, D57, D58, D6, D66, D67, D68, D69, D7: 1N4148, Diode_THT:D_DO-35_SOD27_P7.62mm_Horizontal, symbol Diode:1N4148
- added J1: AudioJack4, Library:TENSILITY_54-00174, symbol Connector_Audio:AudioJack4_SwitchT1
- added SW1, SW16, SW17, SW18, SW19, SW2, SW20, SW3, SW30, SW31, SW32, SW33, SW34, SW4, SW43, SW44, SW45, SW46, SW47, SW5, SW6, SW66, SW67, SW68, SW69, SW7: SW_Push, MX_Hotswap:MX-Hotswap-1U, symbol Switch:SW_Push
- added SW15: SW_Push, MX_Hotswap:MX-Hotswap-1.25U, symbol Switch:SW_Push
- added SW29, SW55, SW56, SW57: SW_Push, MX_Hotswap:MX-Hotswap-1.5U, symbol Switch:SW_Push
- added SW42: SW_Push, MX_Hotswap:MX-Hotswap-1.75U, symbol Switch:SW_Push
- added SW58: SW_Push, MX_Hotswap:MX-Hotswap-2U, symbol Switch:SW_Push
- added U1: ~, Library:SSD1306-0.91-OLED-4pin-128x32, symbol display:.91{dblquote}_4-pin_OLED
Connections:
- new net: A1.2 (GPIO1), SW16.1, SW2.1, SW30.1, SW43.1, SW56.1, SW67.1
- new net: D16.2 (A), SW16.2
- new net: A1.6 (GPIO4), SW19.1, SW33.1, SW46.1, SW5.1
- new net: D19.2 (A), SW19.2
- new net: A1.14 (GPIO10), D42.1 (K), D43.1 (K), D44.1 (K), D45.1 (K), D46.1 (K), D47.1 (K)
- new net: D45.2 (A), SW45.2
- new net: D47.2 (A), SW47.2
- new net: A1.5 (GPIO3), SW18.1, SW32.1, SW4.1, SW45.1, SW58.1, SW69.1
- new net: D4.2 (A), SW4.2
- new net: A1.10 (GPIO7), D1.1 (K), D2.1 (K), D3.1 (K), D4.1 (K), D5.1 (K), D6.1 (K), D7.1 (K)
- new net: A1.7 (GPIO5), SW20.1, SW34.1, SW47.1, SW6.1
- new net: D20.2 (A), SW20.2
- new net: A1.12 (GPIO9), D29.1 (K), D30.1 (K), D31.1 (K), D32.1 (K), D33.1 (K), D34.1 (K)
- new net: D33.2 (A), SW33.2
- new net: D3.2 (A), SW3.2
- new net: D42.2 (A), SW42.2
- new net: D69.2 (A), SW69.2
- new net: A1.9 (GPIO6), SW7.1
- new net: D7.2 (A), SW7.2
- new net: A1.1 (GPIO0), SW1.1, SW15.1, SW29.1, SW42.1, SW55.1, SW66.1
- new net: D55.2 (A), SW55.2
- new net: A1.15 (GPIO11), D55.1 (K), D56.1 (K), D57.1 (K), D58.1 (K)
- new net: D56.2 (A), SW56.2
- new net: D43.2 (A), SW43.2
- new net: A1.4 (GPIO2), SW17.1, SW3.1, SW31.1, SW44.1, SW57.1, SW68.1
- new net: D31.2 (A), SW31.2
- new net: D1.2 (A), SW1.2
- new net: D46.2 (A), SW46.2
- new net: D66.2 (A), SW66.2
- new net: D58.2 (A), SW58.2
- new net: D18.2 (A), SW18.2
- new net: D2.2 (A), SW2.2
- new net: D44.2 (A), SW44.2
- new net: A1.11 (GPIO8), D15.1 (K), D16.1 (K), D17.1 (K), D18.1 (K), D19.1 (K), D20.1 (K)
- new net: D57.2 (A), SW57.2
- new net: A1.16 (GPIO12), D66.1 (K), D67.1 (K), D68.1 (K), D69.1 (K)
- new net: D67.2 (A), SW67.2
- new net: D34.2 (A), SW34.2
- new net: D68.2 (A), SW68.2
- new net: D6.2 (A), SW6.2
- new net: D32.2 (A), SW32.2
- new net: D29.2 (A), SW29.2
- new net: D17.2 (A), SW17.2
- new net: D5.2 (A), SW5.2
- new net: D30.2 (A), SW30.2
- new net: A1.13 (GND), A1.18 (GND), A1.23 (GND), A1.28 (GND), A1.3 (GND), A1.38 (GND), A1.8 (GND), J1.4_1 (T), U1.1 (GND)
- new net: A1.25 (GPIO19), U1.3 (SCL)
- new net: A1.24 (GPIO18), U1.4 (SDA)
- new net: D15.2 (A), SW15.2
- new net: A1.22 (GPIO17), J1.1 (S)
- new net +3.3V: A1.36 (3V3), J1.3 (R1), U1.2 (+5V)
- no-connect marks 30 -> 23
Other:
- added sheet right_side (keyboardv2_right.kicad_sch)
