File: pcb/keyboardv2_right.kicad_sch (KiCad schematic)
At the start: 69 parts, among them J1 AudioJack4, SW1 SW_Push, SW15 SW_Push, SW16 SW_Push, SW17 SW_Push, SW18 SW_Push, SW19 SW_Push, SW2 SW_Push, SW20 SW_Push, SW29 SW_Push, SW3 SW_Push, SW30 SW_Push, SW31 SW_Push, SW32 SW_Push, SW33 SW_Push, SW34 SW_Push, SW4 SW_Push, SW42 SW_Push, SW43 SW_Push, SW44 SW_Push, SW45 SW_Push, SW46 SW_Push, SW47 SW_Push, SW5 SW_Push, SW55 SW_Push, SW56 SW_Push, SW57 SW_Push, SW58 SW_Push, SW6 SW_Push, SW66 SW_Push, SW67 SW_Push, SW68 SW_Push, SW69 SW_Push, SW7 SW_Push

Commit message: bom changes and layout changes
Parts:
- removed A1: RaspberryPi_Pico, Module:RaspberryPi_Pico_Common_THT, symbol MCU_Module_RaspberryPi_Pico:RaspberryPi_Pico
- removed D1, D15, D16, D17, D18, D19, D2, D20, D29, D3, D30, D31, D32, D33, D34, D4, D42, D43, D44, D45, D46, D47, D5, D55, D56, D57, D58, D6, D66, D67, D68, D69, D7: 1N4148, Diode_THT:D_DO-35_SOD27_P7.62mm_Horizontal, symbol Diode:1N4148
- removed J1: AudioJack4, Library:TENSILITY_54-00174, symbol Connector_Audio:AudioJack4_SwitchT1
- removed SW1, SW16, SW17, SW18, SW19, SW2, SW20, SW3, SW30, SW31, SW32, SW33, SW34, SW4, SW43, SW44, SW45, SW46, SW47, SW5, SW6, SW66, SW67, SW68, SW69, SW7: SW_Push, MX_Hotswap:MX-Hotswap-1U, symbol Switch:SW_Push
- removed SW15: SW_Push, MX_Hotswap:MX-Hotswap-1.25U, symbol Switch:SW_Push
- removed SW29, SW55, SW56, SW57: SW_Push, MX_Hotswap:MX-Hotswap-1.5U, symbol Switch:SW_Push
- removed SW42: SW_Push, MX_Hotswap:MX-Hotswap-1.75U, symbol Switch:SW_Push
- removed SW58: SW_Push, MX_Hotswap:MX-Hotswap-2U, symbol Switch:SW_Push
- removed U1: ~, Library:SSD1306-0.91-OLED-4pin-128x32, symbol display:.91{dblquote}_4-pin_OLED
- added A3: RaspberryPi_Pico, Module:RaspberryPi_Pico_Common_THT, symbol MCU_Module_RaspberryPi_Pico:RaspberryPi_Pico
- added D10, D11, D12, D13, D14, D21, D22, D23, D24, D25, D26, D27, D28, D35, D36, D37, D38, D39, D40, D41, D48, D49, D50, D51, D52, D53, D54, D59, D60, D61, D62, D63, D64, D65, D8, D9: 1N4148, Diode_THT:D_DO-35_SOD27_P7.62mm_Horizontal, symbol Diode:1N4148
- added J2: AudioJack4, Library:TENSILITY_54-00174, symbol Connector_Audio:AudioJack4_SwitchT1
- added SW10, SW11, SW12, SW13, SW21, SW22, SW23, SW24, SW25, SW26, SW27, SW28, SW35, SW36, SW37, SW38, SW39, SW40, SW48, SW49, SW50, SW51, SW52, SW54, SW60, SW61, SW62, SW63, SW64, SW65, SW8, SW9: SW_Push, MX_Hotswap:MX-Hotswap-1U, symbol Switch:SW_Push
- added SW14, SW41: SW_Push, MX_Hotswap:MX-Hotswap-1.75U, symbol Switch:SW_Push
- added SW53: SW_Push, MX_Hotswap:MX-Hotswap-1.25U, symbol Switch:SW_Push
- added SW59: SW_Push, MX_Hotswap:MX-Hotswap-2U, symbol Switch:SW_Push
- added U2: ~, Library:SSD1306-0.91-OLED-4pin-128x32, symbol display:.91{dblquote}_4-pin_OLED
Connections:
- new net: A3.16 (GPIO12), D59.1 (K), D60.1 (K), D61.1 (K), D62.1 (K), D63.1 (K), D64.1 (K), D65.1 (K)
- new net: D63.2 (A), SW63.2
- new net: A3.2 (GPIO1), SW22.1, SW36.1, SW49.1, SW60.1, SW8.1
- new net: D49.2 (A), SW49.2
- new net: A3.4 (GPIO2), SW23.1, SW37.1, SW50.1, SW61.1, SW9.1
- new net: D9.2 (A), SW9.2
- new net: A3.14 (GPIO10), D35.1 (K), D36.1 (K), D37.1 (K), D38.1 (K), D39.1 (K), D40.1 (K), D41.1 (K)
- new net: D38.2 (A), SW38.2
- new net: D40.2 (A), SW40.2
- new net: A3.1 (GPIO0), SW21.1, SW35.1, SW48.1, SW59.1
- new net: D21.2 (A), SW21.2
- new net: A3.6 (GPIO4), SW11.1, SW25.1, SW39.1, SW52.1, SW63.1
- new net: D52.2 (A), SW52.2
- new net: A3.7 (GPIO5), SW12.1, SW26.1, SW40.1, SW53.1, SW64.1
- new net: D12.2 (A), SW12.2
- new net: D36.2 (A), SW36.2
- new net: A3.10 (GPIO7), SW14.1, SW28.1
- new net: D14.2 (A), SW14.2
- new net: A3.5 (GPIO3), SW10.1, SW24.1, SW38.1, SW51.1, SW62.1
- new net: A3.15 (GPIO11), D48.1 (K), D49.1 (K), D50.1 (K), D51.1 (K), D52.1 (K), D53.1 (K), D54.1 (K)
- new net: D51.2 (A), SW51.2
- new net: A3.9 (GPIO6), SW13.1, SW27.1, SW41.1, SW54.1, SW65.1
- new net: D54.2 (A), SW54.2
- new net: A3.12 (GPIO9), D21.1 (K), D22.1 (K), D23.1 (K), D24.1 (K), D25.1 (K), D26.1 (K), D27.1 (K), D28.1 (K)
- new net: D25.2 (A), SW25.2
- new net: A3.11 (GPIO8), D10.1 (K), D11.1 (K), D12.1 (K), D13.1 (K), D14.1 (K), D8.1 (K), D9.1 (K)
- new net: D8.2 (A), SW8.2
- new net: D62.2 (A), SW62.2
- new net: D50.2 (A), SW50.2
- new net: D24.2 (A), SW24.2
- new net: D60.2 (A), SW60.2
- new net: D13.2 (A), SW13.2
- new net: D41.2 (A), SW41.2
- new net: D35.2 (A), SW35.2
- new net: D59.2 (A), SW59.2
- new net: D23.2 (A), SW23.2
- new net: D10.2 (A), SW10.2
- new net: D39.2 (A), SW39.2
- new net: D64.2 (A), SW64.2
- new net: D48.2 (A), SW48.2
- new net: D26.2 (A), SW26.2
- new net: D37.2 (A), SW37.2
- new net: D28.2 (A), SW28.2
- new net: D65.2 (A), SW65.2
- new net: A3.22 (GPIO17), J2.1 (S)
- new net: A3.40 (VBUS), J2.3 (R1)
- new net: D61.2 (A), SW61.2
- new net: D53.2 (A), SW53.2
- new net: D11.2 (A), SW11.2
- new net: A3.36 (3V3), U2.2 (+5V)
- new net: A3.25 (GPIO19), U2.3 (SCL)
- new net: A3.24 (GPIO18), U2.4 (SDA)
- new net: D27.2 (A), SW27.2
- new net: D22.2 (A), SW22.2
- new net GND: A3.13 (GND), A3.18 (GND), A3.23 (GND), A3.28 (GND), A3.3 (GND), A3.38 (GND), A3.8 (GND), J2.4_1 (T), U2.1 (GND)
- no-connect marks 23 -> 30
Other:
- removed sheet right_side
