File: pcb/keyboardv2.kicad_pcb (KiCad board)
At the start: 2 copper layers, 364.2 x 100.5 mm, 144 parts, among them J1 AudioJack4, J2 AudioJack4, SW1 SW_Push, SW10 SW_Push, SW11 SW_Push, SW12 SW_Push, SW13 SW_Push, SW14 SW_Push, SW15 SW_Push, SW16 SW_Push, SW17 SW_Push, SW18 SW_Push, SW19 SW_Push, SW2 SW_Push, SW20 SW_Push, SW21 SW_Push, SW22 SW_Push, SW23 SW_Push, SW24 SW_Push, SW25 SW_Push, SW26 SW_Push, SW27 SW_Push, SW28 SW_Push, SW29 SW_Push, SW3 SW_Push, SW30 SW_Push, SW31 SW_Push, SW32 SW_Push, SW33 SW_Push, SW34 SW_Push, SW35 SW_Push, SW36 SW_Push, SW37 SW_Push, SW38 SW_Push, SW39 SW_Push, SW4 SW_Push, SW40 SW_Push, SW41 SW_Push, SW42 SW_Push, SW43 SW_Push, SW44 SW_Push, SW45 SW_Push, SW46 SW_Push, SW47 SW_Push, SW48 SW_Push, SW49 SW_Push, SW5 SW_Push, SW50 SW_Push, SW51 SW_Push, SW52 SW_Push, SW53 SW_Push, SW54 SW_Push, SW55 SW_Push, SW56 SW_Push, SW57 SW_Push, SW58 SW_Push, SW59 SW_Push, SW6 SW_Push, SW60 SW_Push, SW61 SW_Push, SW62 SW_Push, SW63 SW_Push, SW64 SW_Push, SW65 SW_Push, SW66 SW_Push, SW67 SW_Push, SW68 SW_Push, SW69 SW_Push, SW7 SW_Push, SW8 SW_Push, SW9 SW_Push

Commit message: bom changes and layout changes
Other:
- board text added: "PCB3D_BR_a"
- board text added: "PCB3D_BR_b"
- board text added: "PCB3D_TL_a"
- board text added: "PCB3D_TL_b"
Changed lines of the file:
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@@
+		)
+	)
+	(gr_text "PCB3D_TL_a"
+		(at 72.6 64.1 0)
+		(layer "Edge.Cuts")
+		(effects
+			(font
+				(size 1 1)
+				(thickness 0.15)
+			)
+			(justify left bottom)
+		)
+	)
+	(gr_text "PCB3D_BR_a"
+		(at 253.8 164.7 0)
+		(layer "Edge.Cuts")
+		(effects
+			(font
+				(size 1 1)
+				(thickness 0.15)
+			)
+			(justify left bottom)
+		)
+	)
+	(gr_text "PCB3D_BR_b"
+		(at 437.1 164.85 0)
+		(layer "Edge.Cuts")
+		(effects
+			(font
+				(size 1 1)
+				(thickness 0.15)
+			)
+			(justify left bottom)
+		)
+	)
+	(gr_text "PCB3D_TL_b"
+		(at 255.7 64.05 0)
+		(layer "Edge.Cuts")
+		(effects
+			(font
+				(size 1 1)
+				(thickness 0.15)
+			)
+			(justify left bottom)
 		)
 	)

Commit message: working on a full 3d model of the board
Parts:
- A1, A3: footprint Library:RaspberryPi_Pico_Common_THT_wModel -> custom:RaspberryPi_Pico_Common_THT
- J1, J2: footprint Library:TENSILITY_54-00174 -> custom:TENSILITY_54-00174
- SW1, SW10, SW11, SW12, SW13, SW16, SW17, SW18, SW19, SW2, SW20, SW21, SW22, SW23, SW24, SW25, SW26, SW27, SW28, SW3, SW30, SW31, SW32, SW33, SW34, SW35, SW36, SW37, SW38, SW39, SW4, SW40, SW43, SW44, SW45, SW46, SW47, SW48, SW49, SW5, SW50, SW51, SW52, SW54, SW6, SW60, SW61, SW62, SW63, SW64, SW65, SW66, SW67, SW68, SW69, SW7, SW8, SW9: footprint MX_Hotswap:MX-Hotswap-1U -> custom:MX-Hotswap-1U
- SW14, SW41, SW42: footprint MX_Hotswap:MX-Hotswap-1.75U -> custom:MX-Hotswap-1.75U
- SW15, SW53: footprint MX_Hotswap:MX-Hotswap-1.25U -> custom:MX-Hotswap-1.25U
- SW29, SW55, SW56, SW57: footprint MX_Hotswap:MX-Hotswap-1.5U -> custom:MX-Hotswap-1.5U
- SW58, SW59: footprint MX_Hotswap:MX-Hotswap-2U -> custom:MX-Hotswap-2U
- U1, U2: footprint Library:SSD1306-0.91-OLED-4pin-128x32 -> custom:SSD1306-0.91-OLED-4pin-128x32
